File: hardware/keyboard-controller.kicad_sch (KiCad schematic)
At the start: 12 parts, among them J1 Keybed_Connector, U1 Pico, U2 MCP4921, U3 TL431LP, U4 74HC164, U5 74HC164

Commit message: Added voltage regulators and power input to schematic
Parts:
- added C1, C2: (no value), symbol Device:C_Polarized
- added C3, C4: (no value), symbol Device:C
- added J2: (no value), symbol Connector:Barrel_Jack
- added U7: (no value), symbol Regulator_Linear:LM1117-3.3
- added U8: (no value), symbol Regulator_Linear:L78L09_TO92
- R2: value (none) -> 10K
- R3: value (none) -> 22K
- R4: value (none) -> 1K
- U6: value (none) -> LM358
Connections:
- net GND: now also C1.2, C2.2, C3.2, C4.2, J2.2, U7.1 (GND), U8.2 (GND)
- net VSS: now also C2.1, U7.2 (VO); no longer R1.2
- new net +12V: C1.1, C3.1, J2.1, U7.3 (VI), U8.3 (VI)
- new net +9V: C4.1, R1.2, U8.1 (VO)
Other:
- note added: "TODO: Add debug output pins"
- note added: "TODO: filter caps on all ICs"
- note removed: "TODO: Add 12v power source"
- note removed: "TODO: Add 5v regulator"
- note removed: "TODO: filter caps on all ICs TODO: Power rpi TODO: AGND for mcp4921? Check datasheet"
- title: (none) -> Keyboard Controller
