File: hardware/keyboard-controller/power.kicad_sch (KiCad schematic)
At the start: 12 parts, among them J4 Barrel_Jack_Switch, U5 L78L09_TO92, U6 LM358, U7 TL431LP, U8 LM1117-3.3

Commit message: Added footprint for rotary switches
Parts:
- renumbered J4 to J2, R7 to R2, U5 to U3, U6 to U4, U7 to U5, U8 to U6
Changed lines of the file:
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@@
   (junction (at 91.44 62.23) (diameter 0) (color 0 0 0 0)
+  )
+  (junction (at 85.09 73.66) (diameter 0) (color 0 0 0 0)
   )
   (junction (at 191.77 115.57) (diameter 0) (color 0 0 0 0)
@@
     (stroke (width 0) (type default) (color 0 0 0 0))
   )
+  (wire (pts (xy 85.09 73.66) (xy 85.09 77.47))
+    (stroke (width 0) (type default) (color 0 0 0 0))
+  )
   (wire (pts (xy 127 120.65) (xy 127 124.46))
     (stroke (width 0) (type default) (color 0 0 0 0))
@@
     (stroke (width 0) (type default) (color 0 0 0 0))
   )
-  (wire (pts (xy 85.09 69.85) (xy 85.09 71.12))
+  (wire (pts (xy 85.09 69.85) (xy 85.09 73.66))
     (stroke (width 0) (type default) (color 0 0 0 0))
   )
@@
   )
   (wire (pts (xy 85.09 69.85) (xy 91.44 69.85))
+    (stroke (width 0) (type default) (color 0 0 0 0))
+  )
+  (wire (pts (xy 85.09 73.66) (xy 88.9 73.66))
     (stroke (width 0) (type default) (color 0 0 0 0))
   )
@@
   (symbol (lib_id "Amplifier_Operational:LM358") (at 119.38 116.84 0) (unit 3)
     (in_bom yes) (on_board yes) (fields_autoplaced)
-    (property "Reference" "U6" (id 0) (at 118.11 115.5699 0)
+    (property "Reference" "U4" (id 0) (at 118.11 115.5699 0)
       (effects (font (size 1.27 1.27)) (justify left))
     )
@@
   (symbol (lib_id "Device:R") (at 195.58 64.77 270) (unit 1)
     (in_bom yes) (on_board yes) (fields_autoplaced)
-    (property "Reference" "R7" (id 0) (at 195.58 58.42 90))
+    (property "Reference" "R2" (id 0) (at 195.58 58.42 90))
     (property "Value" "100" (id 1) (at 195.58 60.96 90))
     (property "Footprint" "Royal_Ohm_Resistors:R_Axial_DIN0207_L6.8mm_D2.5mm_P10.16mm_Horizontal" (id 2) (at 195.58 62.992 90)
@@
     (pin "2")
   )
-  (symbol (lib_id "power:GND") (at 85.09 71.12 0) (unit 1)
-    (in_bom yes) (on_board yes) (fields_autoplaced)
-    (property "Reference" "#PWR021" (id 0) (at 85.09 77.47 0)
-      (effects (font (size 1.27 1.27)) hide)
-    )
-    (property "Value" "GND" (id 1) (at 85.09 76.2 0))
-    (property "Footprint" "" (id 2) (at 85.09 71.12 0)
-      (effects (font (size 1.27 1.27)) hide)
-    )
-    (property "Datasheet" "" (id 3) (at 85.09 71.12 0)
+  (symbol (lib_id "power:GND") (at 85.09 77.47 0) (unit 1)
+    (in_bom yes) (on_board yes) (fields_autoplaced)
+    (property "Reference" "#PWR022" (id 0) (at 85.09 83.82 0)
+      (effects (font (size 1.27 1.27)) hide)
+    )
+    (property "Value" "GND" (id 1) (at 85.09 82.55 0))
+    (property "Footprint" "" (id 2) (at 85.09 77.47 0)
+      (effects (font (size 1.27 1.27)) hide)
+    )
+    (property "Datasheet" "" (id 3) (at 85.09 77.47 0)
       (effects (font (size 1.27 1.27)) hide)
     )
@@
   (symbol (lib_id "Reference_Voltage:TL431LP") (at 203.2 69.85 90) (unit 1)
     (in_bom yes) (on_board yes) (fields_autoplaced)
-    (property "Reference" "U7" (id 0) (at 205.74 68.5799 90)
+    (property "Reference" "U5" (id 0) (at 205.74 68.5799 90)
       (effects (font (size 1.27 1.27)) (justify right))
     )
@@
   (symbol (lib_id "power:GND") (at 87.63 124.46 0) (unit 1)
     (in_bom yes) (on_board yes) (fields_autoplaced)
-    (property "Reference" "#PWR022" (id 0) (at 87.63 130.81 0)
+    (property "Reference" "#PWR023" (id 0) (at 87.63 130.81 0)
       (effects (font (size 1.27 1.27)) hide)
     )
@@
   (symbol (lib_id "power:GND") (at 208.28 127 0) (unit 1)
     (in_bom yes) (on_board yes) (fields_autoplaced)
-    (property "Reference" "#PWR028" (id 0) (at 208.28 133.35 0)
+    (property "Reference" "#PWR029" (id 0) (at 208.28 133.35 0)
       (effects (font (size 1.27 1.27)) hide)
     )
@@
   (symbol (lib_id "power:+12V") (at 102.87 62.23 0) (unit 1)
     (in_bom yes) (on_board yes) (fields_autoplaced)
-    (property "Reference" "#PWR023" (id 0) (at 102.87 66.04 0)
+    (property "Reference" "#PWR024" (id 0) (at 102.87 66.04 0)
       (effects (font (size 1.27 1.27)) hide)
     )
@@
   (symbol (lib_id "power:+12V") (at 182.88 115.57 0) (unit 1)
     (in_bom yes) (on_board yes) (fields_autoplaced)
-    (property "Reference" "#PWR025" (id 0) (at 182.88 119.38 0)
+    (property "Reference" "#PWR026" (id 0) (at 182.88 119.38 0)
       (effects (font (size 1.27 1.27)) hide)
     )
@@
   (symbol (lib_id "power:PWR_FLAG") (at 208.28 64.77 0) (unit 1)
     (in_bom yes) (on_board yes) (fields_autoplaced)
-    (property "Reference" "#FLG02" (id 0) (at 208.28 62.865 0)
+    (property "Reference" "#FLG03" (id 0) (at 208.28 62.865 0)
       (effects (font (size 1.27 1.27)) hide)
     )
@@
   (symbol (lib_id "power:+12V") (at 62.23 109.22 0) (unit 1)
     (in_bom yes) (on_board yes) (fields_autoplaced)
-    (property "Reference" "#PWR020" (id 0) (at 62.23 113.03 0)
+    (property "Reference" "#PWR021" (id 0) (at 62.23 113.03 0)
       (effects (font (size 1.27 1.27)) hide)
     )
@@
   (symbol (lib_id "power:GND") (at 203.2 73.66 0) (unit 1)
     (in_bom yes) (on_board yes)
-    (property "Reference" "#PWR027" (id 0) (at 203.2 80.01 0)
+    (property "Reference" "#PWR028" (id 0) (at 203.2 80.01 0)
       (effects (font (size 1.27 1.27)) hide)
     )
@@
   (symbol (lib_id "power:+9V") (at 129.54 109.22 0) (unit 1)
     (in_bom yes) (on_board yes) (fields_autoplaced)
-    (property "Reference" "#PWR024" (id 0) (at 129.54 113.03 0)
+    (property "Reference" "#PWR025" (id 0) (at 129.54 113.03 0)
       (effects (font (size 1.27 1.27)) hide)
     )
@@
   (symbol (lib_id "Regulator_Linear:L78L09_TO92") (at 87.63 109.22 0) (unit 1)
     (in_bom yes) (on_board yes)
-    (property "Reference" "U5" (id 0) (at 87.63 101.6 0))
+    (property "Reference" "U3" (id 0) (at 87.63 101.6 0))
     (property "Value" "L78L09_TO92" (id 1) (at 87.63 104.14 0))
     (property "Footprint" "Package_TO_SOT_THT:TO-92_Inline" (id 2) (at 87.63 103.505 0)
@@
   (symbol (lib_id "power:+3.3V") (at 234.95 115.57 0) (unit 1)
     (in_bom yes) (on_board yes) (fields_autoplaced)
-    (property "Reference" "#PWR029" (id 0) (at 234.95 119.38 0)
+    (property "Reference" "#PWR030" (id 0) (at 234.95 119.38 0)
       (effects (font (size 1.27 1.27)) hide)
     )
@@
   (symbol (lib_id "power:+3.3V") (at 186.69 62.23 0) (unit 1)
     (in_bom yes) (on_board yes) (fields_autoplaced)
-    (property "Reference" "#PWR026" (id 0) (at 186.69 66.04 0)
+    (property "Reference" "#PWR027" (id 0) (at 186.69 66.04 0)
       (effects (font (size 1.27 1.27)) hide)
     )
@@
   (symbol (lib_id "Connector:Barrel_Jack_Switch") (at 72.39 64.77 0) (unit 1)
     (in_bom yes) (on_board yes) (fields_autoplaced)
-    (property "Reference" "J4" (id 0) (at 72.39 55.88 0))
+    (property "Reference" "J2" (id 0) (at 72.39 55.88 0))
     (property "Value" "Barrel_Jack_Switch" (id 1) (at 72.39 58.42 0))
     (property "Footprint" "WEALTH_METAL_Barrel_Jacks:BarrelJack_Horizontal_2.1mm_WEALTH_METAL" (id 2) (at 73.66 65.786 0)
@@
   (symbol (lib_id "Regulator_Linear:LM1117-3.3") (at 208.28 115.57 0) (unit 1)
     (in_bom yes) (on_board yes) (fields_autoplaced)
-    (property "Reference" "U8" (id 0) (at 208.28 107.95 0))
+    (property "Reference" "U6" (id 0) (at 208.28 107.95 0))
     (property "Value" "LM1117-3.3" (id 1) (at 208.28 110.49 0))
     (property "Footprint" "Package_TO_SOT_THT:TO-220-3_Horizontal_TabDown" (id 2) (at 208.28 115.57 0)

Commit message: Updated hardware_config and fixed sync_cn
Parts:
- removed C3: 47uF, Capacitor_THT:CP_Radial_D5.0mm_P2.00mm, symbol Device:C_Polarized
- added D6: 1N4001, Diode_THT:D_DO-41_SOD81_P10.16mm_Horizontal, symbol Diode:1N4001
- C5: Notes (none) -> Ceramic
- C6: Notes (none) -> Tantalum
- C7: value 100uF -> 10uF; Notes (none) -> Tantalum
- U4: Supplier (none) -> Tayda
- renumbered C2 to C3, R2 to R6
Connections:
- net +12V: now also D6.1 (K)
- net +9V: now also D6.2 (A)
Other:
- moved on the sheet: C3, C4, C5, U3, U4C
