File: hardware/keyboard-controller/power.kicad_sch (KiCad schematic)
At the start: 10 parts, among them J2 Barrel_Jack_Switch, U3 L78L09_TO92, U4 TL431LP, U5 LM1117-3.3

Commit message: Completed initial pcb design
Connections:
- net +3V3 renamed +3.3V

Commit message: Added more text detail to PCB. Completed more of BOM
Parts:
- C3: Manufacturer (none) -> AVX; Manufacturer Part No. (none) -> 0.33uF 35V Radial Capacitor Tantalum; Notes (none) -> Tantalum; Supplier Part No. (none) -> A-5100
- C4: Manufacturer (none) -> AVX; Manufacturer Part No. (none) -> 0.1uF 35V Radial Capacitor Tantalum; Notes (none) -> Tantalum; Supplier Part No. (none) -> A-1606
- C5, C6: Manufacturer (none) -> AVX; Manufacturer Part No. (none) -> 10uF 35V Radial Capacitor Tantalum; Supplier Part No. (none) -> A-5226
- D6: Manufacturer (none) -> EIC; Manufacturer Part No. (none) -> 1N4001; Supplier Part No. (none) -> A-162
- J2: Manufacturer (none) -> WEALTH METAL; Manufacturer Part No. (none) -> DC Power Jack 2.1mm; Supplier Part No. (none) -> A-4118
- U4: value TL431LP -> TL431; Manufacturer (none) -> VARIOUS; Manufacturer Part No. (none) -> TL431ACL; Supplier (none) -> Tayda; Supplier Part No. (none) -> A-140
Changed lines of the file:
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@@
+      (effects (font (size 1.27 1.27)) hide)
+    )
+    (property "Manufacturer" "AVX" (id 5) (at 66.04 121.92 0)
+      (effects (font (size 1.27 1.27)) hide)
+    )
+    (property "Manufacturer Part No." "0.33uF 35V Radial Capacitor Tantalum" (id 6) (at 66.04 121.92 0)
+      (effects (font (size 1.27 1.27)) hide)
+    )
+    (property "Notes" "Tantalum" (id 7) (at 66.04 121.92 0)
+      (effects (font (size 1.27 1.27)) hide)
+    )
+    (property "Supplier Part No." "A-5100" (id 8) (at 66.04 121.92 0)
       (effects (font (size 1.27 1.27)) hide)
     )
@@
       (effects (font (size 1.27 1.27)) hide)
     )
+    (property "Manufacturer" "EIC" (id 5) (at 82.55 101.6 0)
+      (effects (font (size 1.27 1.27)) hide)
+    )
+    (property "Manufacturer Part No." "1N4001" (id 6) (at 82.55 101.6 0)
+      (effects (font (size 1.27 1.27)) hide)
+    )
+    (property "Supplier Part No." "A-162" (id 7) (at 82.55 101.6 0)
+      (effects (font (size 1.27 1.27)) hide)
+    )
     (pin "1")
     (pin "2")
@@
     )
     (property "Supplier" "Tayda" (id 4) (at 99.06 121.92 0)
+      (effects (font (size 1.27 1.27)) hide)
+    )
+    (property "Manufacturer" "AVX" (id 5) (at 99.06 121.92 0)
+      (effects (font (size 1.27 1.27)) hide)
+    )
+    (property "Manufacturer Part No." "0.1uF 35V Radial Capacitor Tantalum" (id 6) (at 99.06 121.92 0)
+      (effects (font (size 1.27 1.27)) hide)
+    )
+    (property "Notes" "Tantalum" (id 7) (at 99.06 121.92 0)
+      (effects (font (size 1.27 1.27)) hide)
+    )
+    (property "Supplier Part No." "A-1606" (id 8) (at 99.06 121.92 0)
       (effects (font (size 1.27 1.27)) hide)
     )
@@
       (effects (font (size 1.27 1.27)) (justify right))
     )
-    (property "Value" "TL431LP" (id 1) (at 205.74 71.1199 90)
+    (property "Value" "TL431" (id 1) (at 205.74 71.1199 90)
       (effects (font (size 1.27 1.27)) (justify right))
     )
@@
     (property "Datasheet" "http://www.ti.com/lit/ds/symlink/tl431.pdf" (id 3) (at 203.2 69.85 0)
       (effects (font (size 1.27 1.27) italic) hide)
+    )
+    (property "Manufacturer" "VARIOUS" (id 4) (at 203.2 69.85 0)
+      (effects (font (size 1.27 1.27)) hide)
+    )
+    (property "Manufacturer Part No." "TL431ACL" (id 5) (at 203.2 69.85 0)
+      (effects (font (size 1.27 1.27)) hide)
+    )
+    (property "Supplier" "Tayda" (id 6) (at 203.2 69.85 0)
+      (effects (font (size 1.27 1.27)) hide)
+    )
+    (property "Supplier Part No." "A-140" (id 7) (at 203.2 69.85 0)
+      (effects (font (size 1.27 1.27)) hide)
     )
     (pin "1")
@@
       (effects (font (size 1.27 1.27)) hide)
     )
-    (property "Supplier Part No." "" (id 5) (at 224.79 120.65 0)
+    (property "Supplier Part No." "A-5226" (id 5) (at 224.79 120.65 0)
       (effects (font (size 1.27 1.27)) hide)
     )
@@
       (effects (font (size 1.27 1.27)) hide)
     )
+    (property "Manufacturer" "AVX" (id 7) (at 224.79 120.65 0)
+      (effects (font (size 1.27 1.27)) hide)
+    )
+    (property "Manufacturer Part No." "10uF 35V Radial Capacitor Tantalum" (id 8) (at 224.79 120.65 0)
+      (effects (font (size 1.27 1.27)) hide)
+    )
     (pin "1")
     (pin "2")
@@
       (effects (font (size 1.27 1.27)) hide)
     )
-    (property "Supplier Part No." "" (id 5) (at 191.77 120.65 0)
+    (property "Supplier Part No." "A-5226" (id 5) (at 191.77 120.65 0)
       (effects (font (size 1.27 1.27)) hide)
     )
     (property "Notes" "Tantalum" (id 6) (at 191.77 120.65 0)
+      (effects (font (size 1.27 1.27)) hide)
+    )
+    (property "Manufacturer" "AVX" (id 7) (at 191.77 120.65 0)
+      (effects (font (size 1.27 1.27)) hide)
+    )
+    (property "Manufacturer Part No." "10uF 35V Radial Capacitor Tantalum" (id 8) (at 191.77 120.65 0)
       (effects (font (size 1.27 1.27)) hide)
     )
@@
       (effects (font (size 1.27 1.27)) hide)
     )
+    (property "Manufacturer" "WEALTH METAL" (id 5) (at 72.39 64.77 0)
+      (effects (font (size 1.27 1.27)) hide)
+    )
+    (property "Manufacturer Part No." "DC Power Jack 2.1mm" (id 6) (at 72.39 64.77 0)
+      (effects (font (size 1.27 1.27)) hide)
+    )
+    (property "Supplier Part No." "A-4118" (id 7) (at 72.39 64.77 0)
+      (effects (font (size 1.27 1.27)) hide)
+    )

Commit message: Completed BOM
Parts:
- R6: Manufacturer (none) -> Royal Ohm; Manufacturer Part No. (none) -> MF0W4FF1000A50; Supplier Part No. (none) -> A-2245
- U3: Manufacturer (none) -> STMicroelectronics; Manufacturer Part No. (none) -> (none); Notes (none) -> L78L09ACZ; Supplier Part No. (none) -> A-878
- U5: Manufacturer (none) -> National Semiconductors; Manufacturer Part No. (none) -> LM1117T; Supplier Part No. (none) -> A-628
Changed lines of the file:
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@@
+      (effects (font (size 1.27 1.27)) hide)
+    )
+    (property "Manufacturer" "Royal Ohm" (id 5) (at 195.58 64.77 0)
+      (effects (font (size 1.27 1.27)) hide)
+    )
+    (property "Manufacturer Part No." "MF0W4FF1000A50 " (id 6) (at 195.58 64.77 0)
+      (effects (font (size 1.27 1.27)) hide)
+    )
+    (property "Supplier Part No." "A-2245" (id 7) (at 195.58 64.77 0)
       (effects (font (size 1.27 1.27)) hide)
     )
@@
       (effects (font (size 1.27 1.27)) hide)
     )
+    (property "Manufacturer" "STMicroelectronics" (id 5) (at 82.55 116.84 0)
+      (effects (font (size 1.27 1.27)) hide)
+    )
+    (property "Manufacturer Part No." " " (id 6) (at 82.55 116.84 0)
+      (effects (font (size 1.27 1.27)) hide)
+    )
+    (property "Notes" "L78L09ACZ" (id 7) (at 82.55 116.84 0)
+      (effects (font (size 1.27 1.27)) hide)
+    )
+    (property "Supplier Part No." "A-878" (id 8) (at 82.55 116.84 0)
+      (effects (font (size 1.27 1.27)) hide)
+    )
     (pin "1")
     (pin "2")
@@
       (effects (font (size 1.27 1.27)) hide)
     )
+    (property "Manufacturer" "National Semiconductors" (id 5) (at 208.28 115.57 0)
+      (effects (font (size 1.27 1.27)) hide)
+    )
+    (property "Manufacturer Part No." "LM1117T" (id 6) (at 208.28 115.57 0)
+      (effects (font (size 1.27 1.27)) hide)
+    )
+    (property "Supplier Part No." "A-628" (id 7) (at 208.28 115.57 0)
+      (effects (font (size 1.27 1.27)) hide)
+    )
