File: hardware/keyboard-controller/keyboard-controller.kicad_pcb (KiCad board)
At the start: 2 copper layers, 257 x 195 mm, 118 parts, among them J1 Debug_Pins, J2 Barrel_Jack_Switch, J3 Keybed Connector, J4 SYNC_IN, J5 CV_OUT, J6 GATE_OUT, J7 SYNC_OUT, Q1 2N3904, SW1 RESET, SW10 FUNCTION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

Commit message: Added more text detail to PCB. Completed more of BOM
Parts:
- added REF**: Polarity_Center_Positive_6mm_SilkScreen, Symbol:Polarity_Center_Positive_6mm_SilkScreen, F.Cu at (333.2, 155.7)
Other:
- board text added: "12V, 200mA"
- board text added: "Clock Division"
- board text added: "July, 2022"
- board text added: "Keyboard Controller - REV1"
- board text added: "Mode"
- board text added: "Northridge Devices"
- board text added: "Reset"
- board text removed: "Keyboard Controller Rev1"

Commit message: Cleaned up tracks
Routing:
- net /MATRIX_R5: track 114.9 -> 130.1 mm
- net /MATRIX_R6: track 118.8 -> 133.4 mm
- net /MATRIX_R4: track 110.7 -> 121.2 mm
- net /MATRIX_DATA: track 145.7 -> 136.8 mm
- net Net-(D7-Pad1): track 46.1 -> 40.5 mm
- net /MATRIX_R1: track 90.9 -> 95.2 mm
- net /MATRIX_R2: track 98.6 -> 100.3 mm
