File: hardware/keyboard-controller/analog_input.kicad_sch (KiCad schematic)
At the start: 41 parts

Commit message: Added footprint for rotary switches
Parts:
- SW11, SW12: renamed from SW?; footprint (none) -> SamacSys_Parts:SR2612F011221R0BD8N; Manufacturer (none) -> Alpha; Manufacturer Part No. (none) -> SR2612F-0112-38F5B-D8-S; Supplier Tayda -> Mouser; Supplier Part No. (none) -> 105-SR2612F-12-38S
- gave numbers to parts that had none: 39

Commit message: Updated hardware_config and fixed sync_cn
Parts:
- C10, C11, C12, C13, C14, C15, C16, C17, C18, C19, C20: Notes (none) -> Ceramic
- U10: Supplier (none) -> Tayda
- renumbered R14 to R19, R15 to R20, R16 to R21, R17 to R22, R18 to R23, R19 to R24, R20 to R25, R21 to R26, R22 to R27, R23 to R28, R24 to R29, R25 to R30, R26 to R31, R27 to R32, R28 to R33, R29 to R34, R30 to R35, R31 to R36, R32 to R37, R33 to R38, R34 to R39, R35 to R40, R36 to R41, R37 to R42

Commit message: Completed schematic rev1. Started placing pcb
Parts:
- R19, R20, R21, R22, R23, R24, R25, R26, R27, R28, R29, R30, R31, R32, R33, R34, R35, R36, R37, R38, R39, R40, R41, R42: footprint (none) -> Royal_Ohm_Resistors:R_Axial_DIN0207_L6.8mm_D2.5mm_P10.16mm_Horizontal
- RV1, RV2, RV3: footprint (none) -> Alpha_Potentiometers:Potentiometer_Alpha_RV09AF-40-20K-B1K_Single_Vertical
- SW11, SW12: Manufacturer Alpha -> (none); Manufacturer Part No. SR2612F-0112-38F5B-D8-S -> (none); Supplier Mouser -> (none); Supplier Part No. 105-SR2612F-12-38S -> (none)
- U9: renamed from U10; footprint (none) -> Package_DIP:DIP-16_W7.62mm_Socket
Other:
- title: (none) -> Analog Input

Commit message: Completed initial pcb design
Parts:
- SW11: footprint SamacSys_Parts:SR2612F011221R0BD8N -> Keyboard:Clock_Div_Switch
- SW12: footprint SamacSys_Parts:SR2612F011221R0BD8N -> Keyboard:Sub_Mode_Switch
- renumbered C10 to C11, C11 to C12, C12 to C13, C13 to C14, C14 to C15, C15 to C16, C16 to C17, C17 to C18, C18 to C19, C19 to C20, C20 to C21, R19 to R21, R20 to R22, R21 to R23, R22 to R24, R23 to R25, R24 to R26, R25 to R27, R26 to R28, R27 to R29, R28 to R30, R29 to R31, R30 to R32, R31 to R33, R32 to R34, R33 to R35, R34 to R36, R35 to R37, R36 to R38, R37 to R39, R38 to R40, R39 to R41, R40 to R42, R41 to R43, R42 to R44, U9 to U10
Connections:
- net CLK_SPEED: now also U10.15 (X2); no longer U10.13 (X0)
- net GATE_TIME: now also U10.13 (X0); no longer U10.15 (X2)
- net +3V3 renamed +3.3V

Commit message: Completed BOM
Parts:
- R21, R22, R23, R24, R25, R26, R27, R28, R29, R30, R31, R32, R33, R34, R35, R36, R37, R38, R39, R40, R41, R42, R43, R44: Manufacturer (none) -> Royal Ohm; Manufacturer Part No. (none) -> MF0W4FF2201A50; Supplier Part No. (none) -> A-2341
- RV1, RV2, RV3: Manufacturer (none) -> ALPHA; Manufacturer Part No. (none) -> RV09AF-40-20K-B100K; Supplier Part No. (none) -> A-1851
- SW11, SW12: Manufacturer (none) -> Alpha; Manufacturer Part No. (none) -> SR2612F-0112-38F5B-D8-S; Supplier (none) -> Mouser; Supplier Part No. (none) -> 105-SR2612F-12-38S
- U10: Manufacturer (none) -> VARIOUS; Manufacturer Part No. (none) -> CD4051BE; Supplier Part No. (none) -> A-495
