File: hardware/keyboard-controller/input_output.kicad_sch (KiCad schematic)
At the start: 25 parts, among them J4 SYNC_IN, J5 CV_OUT, J6 GATE_OUT, J7 SYNC_OUT, Q1 2N3904, U8 LM358, U9 LM358

Commit message: Completed BOM
Parts:
- R10, R9: Manufacturer (none) -> Royal Ohm; Manufacturer Part No. (none) -> MF0W4FF1004A50; Supplier Part No. (none) -> A-2277
- R11: value 1k -> 1K; Manufacturer (none) -> Royal Ohm; Manufacturer Part No. (none) -> MF0W4FF1001A50; Supplier Part No. (none) -> A-2200
- R12, R15, R17: Manufacturer (none) -> Royal Ohm; Manufacturer Part No. (none) -> MF0W4FF1002A50; Supplier Part No. (none) -> A-2203
- R13, R14: Manufacturer (none) -> Royal Ohm; Manufacturer Part No. (none) -> MF0W4FF2002A50; Supplier Part No. (none) -> A-2339
- R16: Manufacturer (none) -> Royal Ohm; Manufacturer Part No. (none) -> MF0W4FF2202A50; Supplier Part No. (none) -> A-2284
- R18, R19, R20, R7: Manufacturer (none) -> Royal Ohm; Manufacturer Part No. (none) -> MF0W4FF1001A50; Supplier Part No. (none) -> A-2200
- R8: Manufacturer (none) -> Royal Ohm; Manufacturer Part No. (none) -> MF0W4FF1003A50; Supplier Part No. (none) -> A-2248
- U8, U9: Manufacturer (none) -> VARIOUS; Manufacturer Part No. (none) -> LM358P; Supplier Part No. (none) -> A-045
Changed lines of the file:
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@@
+      (effects (font (size 1.27 1.27)) hide)
+    )
+    (property "Manufacturer" "Royal Ohm" (id 5) (at 59.69 66.04 0)
+      (effects (font (size 1.27 1.27)) hide)
+    )
+    (property "Supplier Part No." "A-2200" (id 6) (at 59.69 66.04 0)
+      (effects (font (size 1.27 1.27)) hide)
+    )
+    (property "Manufacturer Part No." "MF0W4FF1001A50" (id 7) (at 59.69 66.04 0)
       (effects (font (size 1.27 1.27)) hide)
     )
@@
       (effects (font (size 1.27 1.27)) hide)
     )
+    (property "Manufacturer" "Royal Ohm" (id 5) (at 74.93 99.06 0)
+      (effects (font (size 1.27 1.27)) hide)
+    )
+    (property "Manufacturer Part No." "MF0W4FF1004A50" (id 6) (at 74.93 99.06 0)
+      (effects (font (size 1.27 1.27)) hide)
+    )
+    (property "Supplier Part No." "A-2277" (id 7) (at 74.93 99.06 0)
+      (effects (font (size 1.27 1.27)) hide)
+    )
     (pin "1")
     (pin "2")
@@
       (effects (font (size 1.27 1.27)) hide)
     )
+    (property "Manufacturer" "Royal Ohm" (id 5) (at 196.85 132.08 0)
+      (effects (font (size 1.27 1.27)) hide)
+    )
+    (property "Manufacturer Part No." "MF0W4FF2002A50" (id 6) (at 196.85 132.08 0)
+      (effects (font (size 1.27 1.27)) hide)
+    )
+    (property "Supplier Part No." "A-2339" (id 7) (at 196.85 132.08 0)
+      (effects (font (size 1.27 1.27)) hide)
+    )
     (pin "1")
     (pin "2")
@@
       (effects (font (size 1.27 1.27)) (justify left))
     )
-    (property "Value" "1k" (id 1) (at 95.25 82.5499 0)
+    (property "Value" "1K" (id 1) (at 95.25 82.5499 0)
       (effects (font (size 1.27 1.27)) (justify left))
     )
@@
     )
     (property "Supplier" "Tayda" (id 4) (at 92.71 81.28 0)
+      (effects (font (size 1.27 1.27)) hide)
+    )
+    (property "Manufacturer" "Royal Ohm" (id 5) (at 92.71 81.28 0)
+      (effects (font (size 1.27 1.27)) hide)
+    )
+    (property "Manufacturer Part No." "MF0W4FF1001A50" (id 6) (at 92.71 81.28 0)
+      (effects (font (size 1.27 1.27)) hide)
+    )
+    (property "Supplier Part No." "A-2200" (id 7) (at 92.71 81.28 0)
       (effects (font (size 1.27 1.27)) hide)
     )
@@
       (effects (font (size 1.27 1.27)) hide)
     )
+    (property "Manufacturer" "Royal Ohm" (id 5) (at 219.71 69.85 0)
+      (effects (font (size 1.27 1.27)) hide)
+    )
+    (property "Supplier Part No." "A-2200" (id 6) (at 219.71 69.85 0)
+      (effects (font (size 1.27 1.27)) hide)
+    )
+    (property "Manufacturer Part No." "MF0W4FF1001A50" (id 7) (at 219.71 69.85 0)
+      (effects (font (size 1.27 1.27)) hide)
+    )
     (pin "1")
     (pin "2")
@@
     )
     (property "Supplier" "Tayda" (id 4) (at 97.79 167.64 0)
+      (effects (font (size 1.27 1.27)) hide)
+    )
+    (property "Manufacturer" "VARIOUS" (id 5) (at 97.79 167.64 0)
+      (effects (font (size 1.27 1.27)) hide)
+    )
+    (property "Manufacturer Part No." "LM358P" (id 6) (at 97.79 167.64 0)
+      (effects (font (size 1.27 1.27)) hide)
+    )
+    (property "Supplier Part No." "A-045" (id 7) (at 97.79 167.64 0)
       (effects (font (size 1.27 1.27)) hide)
     )
@@
       (effects (font (size 1.27 1.27)) hide)
     )
+    (property "Manufacturer" "Royal Ohm" (id 5) (at 207.01 80.01 0)
+      (effects (font (size 1.27 1.27)) hide)
+    )
+    (property "Manufacturer Part No." "MF0W4FF1002A50" (id 6) (at 207.01 80.01 0)
+      (effects (font (size 1.27 1.27)) hide)
+    )
+    (property "Supplier Part No." "A-2203" (id 7) (at 207.01 80.01 0)
+      (effects (font (size 1.27 1.27)) hide)
+    )
     (pin "1")
     (pin "2")
@@
       (effects (font (size 1.27 1.27)) hide)
     )
+    (property "Manufacturer" "Royal Ohm" (id 5) (at 208.28 38.1 0)
+      (effects (font (size 1.27 1.27)) hide)
+    )
+    (property "Manufacturer Part No." "MF0W4FF2202A50" (id 6) (at 208.28 38.1 0)
+      (effects (font (size 1.27 1.27)) hide)
+    )
+    (property "Supplier Part No." "A-2284" (id 7) (at 208.28 38.1 0)
+      (effects (font (size 1.27 1.27)) hide)
+    )
     (pin "1")
     (pin "2")
@@
       (effects (font (size 1.27 1.27)) hide)
     )
+    (property "Manufacturer" "Royal Ohm" (id 5) (at 208.28 128.27 0)
+      (effects (font (size 1.27 1.27)) hide)
+    )
+    (property "Manufacturer Part No." "MF0W4FF1002A50" (id 6) (at 208.28 128.27 0)
+      (effects (font (size 1.27 1.27)) hide)
+    )
+    (property "Supplier Part No." "A-2203" (id 7) (at 208.28 128.27 0)
+      (effects (font (size 1.27 1.27)) hide)
+    )
     (pin "1")
     (pin "2")
@@
     )
     (property "Supplier" "Tayda" (id 4) (at 146.05 170.18 0)
+      (effects (font (size 1.27 1.27)) hide)
+    )
+    (property "Manufacturer" "VARIOUS" (id 5) (at 146.05 170.18 0)
+      (effects (font (size 1.27 1.27)) hide)
+    )
+    (property "Manufacturer Part No." "LM358P" (id 6) (at 146.05 170.18 0)
+      (effects (font (size 1.27 1.27)) hide)
+    )
+    (property "Supplier Part No." "A-045" (id 7) (at 146.05 170.18 0)
       (effects (font (size 1.27 1.27)) hide)
     )
@@
       (effects (font (size 1.27 1.27)) hide)
     )
+    (property "Manufacturer" "Royal Ohm" (id 5) (at 195.58 41.91 0)
+      (effects (font (size 1.27 1.27)) hide)
+    )
+    (property "Manufacturer Part No." "MF0W4FF1002A50" (id 6) (at 195.58 41.91 0)
+      (effects (font (size 1.27 1.27)) hide)
+    )
+    (property "Supplier Part No." "A-2203" (id 7) (at 195.58 41.91 0)
+      (effects (font (size 1.27 1.27)) hide)
+    )
     (pin "1")
     (pin "2")
@@
       (effects (font (size 1.27 1.27)) hide)
     )
+    (property "Manufacturer" "Royal Ohm" (id 5) (at 66.04 92.71 0)
+      (effects (font (size 1.27 1.27)) hide)
+    )
+    (property "Manufacturer Part No." "MF0W4FF1003A50" (id 6) (at 66.04 92.71 0)
+      (effects (font (size 1.27 1.27)) hide)
+    )
+    (property "Supplier Part No." "A-2248" (id 7) (at 66.04 92.71 0)
+      (effects (font (size 1.27 1.27)) hide)
+    )
     (pin "1")
     (pin "2")
@@
     )
     (property "Supplier" "Tayda" (id 4) (at 135.89 170.18 0)
+      (effects (font (size 1.27 1.27)) hide)
+    )
+    (property "Manufacturer" "VARIOUS" (id 5) (at 135.89 170.18 0)
+      (effects (font (size 1.27 1.27)) hide)
+    )
+    (property "Manufacturer Part No." "LM358P" (id 6) (at 135.89 170.18 0)
+      (effects (font (size 1.27 1.27)) hide)
+    )
+    (property "Supplier Part No." "A-045" (id 7) (at 135.89 170.18 0)
       (effects (font (size 1.27 1.27)) hide)
     )
@@
       (effects (font (size 1.27 1.27)) hide)
     )
+    (property "Manufacturer" "Royal Ohm" (id 5) (at 219.71 27.94 0)
+      (effects (font (size 1.27 1.27)) hide)
+    )
+    (property "Supplier Part No." "A-2200" (id 6) (at 219.71 27.94 0)
+      (effects (font (size 1.27 1.27)) hide)
+    )
+    (property "Manufacturer Part No." "MF0W4FF1001A50" (id 7) (at 219.71 27.94 0)
+      (effects (font (size 1.27 1.27)) hide)
+    )
     (pin "1")
     (pin "2")
@@
       (effects (font (size 1.27 1.27)) hide)
     )
+    (property "Manufacturer" "Royal Ohm" (id 5) (at 220.98 118.11 0)
+      (effects (font (size 1.27 1.27)) hide)
+    )
+    (property "Supplier Part No." "A-2200" (id 6) (at 220.98 118.11 0)
+      (effects (font (size 1.27 1.27)) hide)
+    )
+    (property "Manufacturer Part No." "MF0W4FF1001A50" (id 7) (at 220.98 118.11 0)
+      (effects (font (size 1.27 1.27)) hide)
+    )
     (pin "1")
     (pin "2")
@@
     )
     (property "Supplier" "Tayda" (id 4) (at 204.47 69.85 0)
+      (effects (font (size 1.27 1.27)) hide)
+    )
+    (property "Manufacturer" "VARIOUS" (id 5) (at 204.47 69.85 0)
+      (effects (font (size 1.27 1.27)) hide)
+    )
+    (property "Manufacturer Part No." "LM358P" (id 6) (at 204.47 69.85 0)
+      (effects (font (size 1.27 1.27)) hide)
+    )
+    (property "Supplier Part No." "A-045" (id 7) (at 204.47 69.85 0)
       (effects (font (size 1.27 1.27)) hide)
     )
@@
       (effects (font (size 1.27 1.27)) hide)
     )
+    (property "Manufacturer" "VARIOUS" (id 5) (at 205.74 118.11 0)
+      (effects (font (size 1.27 1.27)) hide)
+    )
+    (property "Manufacturer Part No." "LM358P" (id 6) (at 205.74 118.11 0)
+      (effects (font (size 1.27 1.27)) hide)
+    )
+    (property "Supplier Part No." "A-045" (id 7) (at 205.74 118.11 0)
+      (effects (font (size 1.27 1.27)) hide)
+    )
     (pin "1")
     (pin "2")
@@
       (effects (font (size 1.27 1.27)) hide)
     )
+    (property "Manufacturer" "Royal Ohm" (id 5) (at 195.58 83.82 0)
+      (effects (font (size 1.27 1.27)) hide)
+    )
+    (property "Manufacturer Part No." "MF0W4FF2002A50" (id 6) (at 195.58 83.82 0)
+      (effects (font (size 1.27 1.27)) hide)
+    )
+    (property "Supplier Part No." "A-2339" (id 7) (at 195.58 83.82 0)
+      (effects (font (size 1.27 1.27)) hide)
+    )
     (pin "1")
     (pin "2")
@@
     )
     (property "Supplier" "Tayda" (id 4) (at 86.36 59.69 0)
+      (effects (font (size 1.27 1.27)) hide)
+    )
+    (property "Manufacturer" "Royal Ohm" (id 5) (at 86.36 59.69 0)
+      (effects (font (size 1.27 1.27)) hide)
+    )
+    (property "Manufacturer Part No." "MF0W4FF1004A50" (id 6) (at 86.36 59.69 0)
+      (effects (font (size 1.27 1.27)) hide)
+    )
+    (property "Supplier Part No." "A-2277" (id 7) (at 86.36 59.69 0)
       (effects (font (size 1.27 1.27)) hide)
     )
@@
       (effects (font (size 1.27 1.27)) hide)
     )
+    (property "Manufacturer" "VARIOUS" (id 5) (at 204.47 27.94 0)
+      (effects (font (size 1.27 1.27)) hide)
+    )
+    (property "Manufacturer Part No." "LM358P" (id 6) (at 204.47 27.94 0)
+      (effects (font (size 1.27 1.27)) hide)
+    )
+    (property "Supplier Part No." "A-045" (id 7) (at 204.47 27.94 0)
+      (effects (font (size 1.27 1.27)) hide)
+    )
