File: hardware/keyboard-controller/key_matrix.kicad_sch (KiCad schematic)
At the start: 21 parts, among them J3 Keybed Connector, SW10 REST, SW3 OCTAVE_UP, SW4 OCTAVE_DOWN, SW5 PLAY_PAUSE, SW6 STOP, SW7 RECORD, SW8 HOLD, SW9 FUNC, U6 74HC164, U7 74HC164

Commit message: Added more text detail to PCB. Completed more of BOM
Parts:
- D10, D11, D12, D13, D14, D7, D8, D9: Manufacturer (none) -> PHILIPS/NXP/ON SEMICONDUCTOR//TAK CHEONG; Manufacturer Part No. (none) -> 1N4148; Supplier Part No. (none) -> A-157
- J3: Manufacturer (none) -> TAIWAN; Manufacturer Part No. (none) -> BHD16PHZT; Supplier (none) -> Tayda; Supplier Part No. (none) -> A-2956
Changed lines of the file:
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@@
+      (effects (font (size 1.27 1.27)) hide)
+    )
+    (property "Manufacturer" "PHILIPS/NXP/ON SEMICONDUCTOR//TAK CHEONG" (id 5) (at 139.7 127 0)
+      (effects (font (size 1.27 1.27)) hide)
+    )
+    (property "Manufacturer Part No." "1N4148" (id 6) (at 139.7 127 0)
+      (effects (font (size 1.27 1.27)) hide)
+    )
+    (property "Supplier Part No." "A-157" (id 7) (at 139.7 127 0)
       (effects (font (size 1.27 1.27)) hide)
     )
@@
       (effects (font (size 1.27 1.27)) hide)
     )
+    (property "Manufacturer" "PHILIPS/NXP/ON SEMICONDUCTOR//TAK CHEONG" (id 5) (at 139.7 90.17 0)
+      (effects (font (size 1.27 1.27)) hide)
+    )
+    (property "Manufacturer Part No." "1N4148" (id 6) (at 139.7 90.17 0)
+      (effects (font (size 1.27 1.27)) hide)
+    )
+    (property "Supplier Part No." "A-157" (id 7) (at 139.7 90.17 0)
+      (effects (font (size 1.27 1.27)) hide)
+    )
     (pin "1")
     (pin "2")
@@
       (effects (font (size 1.27 1.27)) hide)
     )
+    (property "Manufacturer" "PHILIPS/NXP/ON SEMICONDUCTOR//TAK CHEONG" (id 5) (at 139.7 52.07 0)
+      (effects (font (size 1.27 1.27)) hide)
+    )
+    (property "Manufacturer Part No." "1N4148" (id 6) (at 139.7 52.07 0)
+      (effects (font (size 1.27 1.27)) hide)
+    )
+    (property "Supplier Part No." "A-157" (id 7) (at 139.7 52.07 0)
+      (effects (font (size 1.27 1.27)) hide)
+    )
     (pin "1")
     (pin "2")
@@
       (effects (font (size 1.27 1.27)) hide)
     )
+    (property "Manufacturer" "PHILIPS/NXP/ON SEMICONDUCTOR//TAK CHEONG" (id 5) (at 139.7 64.77 0)
+      (effects (font (size 1.27 1.27)) hide)
+    )
+    (property "Manufacturer Part No." "1N4148" (id 6) (at 139.7 64.77 0)
+      (effects (font (size 1.27 1.27)) hide)
+    )
+    (property "Supplier Part No." "A-157" (id 7) (at 139.7 64.77 0)
+      (effects (font (size 1.27 1.27)) hide)
+    )
     (pin "1")
     (pin "2")
@@
       (effects (font (size 1.27 1.27)) hide)
     )
+    (property "Manufacturer" "PHILIPS/NXP/ON SEMICONDUCTOR//TAK CHEONG" (id 5) (at 139.7 102.87 0)
+      (effects (font (size 1.27 1.27)) hide)
+    )
+    (property "Manufacturer Part No." "1N4148" (id 6) (at 139.7 102.87 0)
+      (effects (font (size 1.27 1.27)) hide)
+    )
+    (property "Supplier Part No." "A-157" (id 7) (at 139.7 102.87 0)
+      (effects (font (size 1.27 1.27)) hide)
+    )
     (pin "1")
     (pin "2")
@@
       (effects (font (size 1.27 1.27)) hide)
     )
+    (property "Manufacturer" "PHILIPS/NXP/ON SEMICONDUCTOR//TAK CHEONG" (id 5) (at 139.7 139.7 0)
+      (effects (font (size 1.27 1.27)) hide)
+    )
+    (property "Manufacturer Part No." "1N4148" (id 6) (at 139.7 139.7 0)
+      (effects (font (size 1.27 1.27)) hide)
+    )
+    (property "Supplier Part No." "A-157" (id 7) (at 139.7 139.7 0)
+      (effects (font (size 1.27 1.27)) hide)
+    )
     (pin "1")
     (pin "2")
@@
     )
     (property "Datasheet" "~" (id 3) (at 72.39 67.31 0)
+      (effects (font (size 1.27 1.27)) hide)
+    )
+    (property "Supplier" "Tayda" (id 4) (at 72.39 67.31 0)
+      (effects (font (size 1.27 1.27)) hide)
+    )
+    (property "Manufacturer" "TAIWAN" (id 5) (at 72.39 67.31 0)
+      (effects (font (size 1.27 1.27)) hide)
+    )
+    (property "Manufacturer Part No." "BHD16PHZT" (id 6) (at 72.39 67.31 0)
+      (effects (font (size 1.27 1.27)) hide)
+    )
+    (property "Supplier Part No." "A-2956" (id 7) (at 72.39 67.31 0)
       (effects (font (size 1.27 1.27)) hide)
     )
@@
       (effects (font (size 1.27 1.27)) hide)
     )
+    (property "Manufacturer" "PHILIPS/NXP/ON SEMICONDUCTOR//TAK CHEONG" (id 5) (at 139.7 114.3 0)
+      (effects (font (size 1.27 1.27)) hide)
+    )
+    (property "Manufacturer Part No." "1N4148" (id 6) (at 139.7 114.3 0)
+      (effects (font (size 1.27 1.27)) hide)
+    )
+    (property "Supplier Part No." "A-157" (id 7) (at 139.7 114.3 0)
+      (effects (font (size 1.27 1.27)) hide)
+    )
     (pin "1")
     (pin "2")
@@
       (effects (font (size 1.27 1.27)) hide)
     )
+    (property "Manufacturer" "PHILIPS/NXP/ON SEMICONDUCTOR//TAK CHEONG" (id 5) (at 139.7 77.47 0)
+      (effects (font (size 1.27 1.27)) hide)
+    )
+    (property "Manufacturer Part No." "1N4148" (id 6) (at 139.7 77.47 0)
+      (effects (font (size 1.27 1.27)) hide)
+    )
+    (property "Supplier Part No." "A-157" (id 7) (at 139.7 77.47 0)
+      (effects (font (size 1.27 1.27)) hide)
+    )

Commit message: Completed BOM
Parts:
- U6, U7: Manufacturer (none) -> VARIOUS; Manufacturer Part No. (none) -> SN74HC164N; Supplier Part No. (none) -> A-922
Changed lines of the file:
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@@
+      (effects (font (size 1.27 1.27)) hide)
+    )
+    (property "Manufacturer" "VARIOUS" (id 5) (at 215.9 111.76 0)
+      (effects (font (size 1.27 1.27)) hide)
+    )
+    (property "Manufacturer Part No." "SN74HC164N" (id 6) (at 215.9 111.76 0)
+      (effects (font (size 1.27 1.27)) hide)
+    )
+    (property "Supplier Part No." "A-922" (id 7) (at 215.9 111.76 0)
       (effects (font (size 1.27 1.27)) hide)
     )
@@
       (effects (font (size 1.27 1.27)) hide)
     )
+    (property "Manufacturer" "VARIOUS" (id 5) (at 215.9 66.04 0)
+      (effects (font (size 1.27 1.27)) hide)
+    )
+    (property "Manufacturer Part No." "SN74HC164N" (id 6) (at 215.9 66.04 0)
+      (effects (font (size 1.27 1.27)) hide)
+    )
+    (property "Supplier Part No." "A-922" (id 7) (at 215.9 66.04 0)
+      (effects (font (size 1.27 1.27)) hide)
+    )
